File: pcb/AS5047-DevBoard/AS5047-Devboard/AS5047-Devboard.kicad_pcb (KiCad board)
At the start: 2 copper layers, 42 x 42 mm, 8 parts, among them J1 SPI_CONN, U1 AS5047P

Commit message: updated ground pour
Other:
- outline, holes or cut-outs redrawn
Changed lines of the file:
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@@
+		(layer "Dwgs.User")
+	)
+	(gr_line
+		(start 134.9 84.65)
+		(end 139.1 84.65)
+		(stroke
+			(width 0.1)
+			(type dot)
+		)
+		(layer "Dwgs.User")
+	)
+	(gr_line
+		(start 134.9 84.65)
+		(end 134.9 88.85)
+		(stroke
+			(width 0.1)
+			(type dot)
+		)
 		(layer "Dwgs.User")
 	)
@@
 	)
 	(gr_line
-		(start 176.9 84.65)
-		(end 134.9 84.65)
-		(stroke
-			(width 0.1)
-			(type solid)
-		)
-		(layer "Edge.Cuts")
-	)
-	(gr_line
-		(start 176.9 126.65)
-		(end 134.9 126.65)
-		(stroke
-			(width 0.1)
-			(type solid)
-		)
-		(layer "Edge.Cuts")
-	)
-	(gr_line
-		(start 134.9 126.65)
-		(end 134.9 84.65)
-		(stroke
-			(width 0.1)
-			(type solid)
-		)
-		(layer "Edge.Cuts")
-	)
-	(gr_line
-		(start 176.9 84.65)
-		(end 176.9 126.65)
+		(start 176.9 122.45)
+		(end 172.7 126.65)
+		(stroke
+			(width 0.1)
+			(type solid)
+		)
+		(layer "Edge.Cuts")
+	)
+	(gr_line
+		(start 176.9 88.85)
+		(end 172.7 84.65)
+		(stroke
+			(width 0.1)
+			(type solid)
+		)
+		(layer "Edge.Cuts")
+	)
+	(gr_line
+		(start 172.7 84.65)
+		(end 139.1 84.65)
+		(stroke
+			(width 0.1)
+			(type solid)
+		)
+		(layer "Edge.Cuts")
+	)
+	(gr_line
+		(start 172.7 126.65)
+		(end 139.1 126.65)
+		(stroke
+			(width 0.1)
+			(type solid)
+		)
+		(layer "Edge.Cuts")
+	)
+	(gr_line
+		(start 134.9 88.85)
+		(end 139.1 84.65)
+		(stroke
+			(width 0.1)
+			(type solid)
+		)
+		(layer "Edge.Cuts")
+	)
+	(gr_line
+		(start 134.9 122.45)
+		(end 134.9 88.85)
+		(stroke
+			(width 0.1)
+			(type solid)
+		)
+		(layer "Edge.Cuts")
+	)
+	(gr_line
+		(start 134.9 122.45)
+		(end 139.1 126.65)
+		(stroke
+			(width 0.1)
+			(type solid)
+		)
+		(layer "Edge.Cuts")
+	)
+	(gr_line
+		(start 176.9 88.85)
+		(end 176.9 122.45)
 		(stroke
 			(width 0.1)
@@
 	)
 	(zone
+		(net 0)
+		(net_name "")
+		(layer "F.Cu")
+		(name "GND")
+		(hatch edge 0.5)
+		(connect_pads
+			(clearance 0)
+		)
+		(min_thickness 0.25)
+		(filled_areas_thickness no)
+		(keepout
+			(tracks not_allowed)
+			(vias not_allowed)
+			(pads not_allowed)
+			(copperpour not_allowed)
+			(footprints allowed)
+		)
+		(placement
+			(enabled no)
+			(sheetname "")
+		)
+		(fill
+			(thermal_gap 0.5)
+			(thermal_bridge_width 0.5)
+		)
+		(polygon
+			(pts
+				(xy 159.45 104.2) (xy 160.25 104.05) (xy 160.5 104.75) (xy 159.45 104.7)
+			)
+		)
+	)
+	(zone
