File: pcb/AS5047-Devboard/AS5047-Devboard.kicad_sch (KiCad schematic)
At the start: 7 parts, among them J1 SPI_CONN, U1 AS5047P

Commit message: updated BOM
Parts:
- C1: JLCPCB Part # C1592 -> C15849
Changed lines of the file:
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@@
 			)
 		)
-		(property "JLCPCB Part #" "C1592"
+		(property "JLCPCB Part #" "C15849"
 			(at 116.84 101.6 0)
 			(effects
