File: pcb/DRV8874-Devboard/_autosave-DRV8874-Devboard.kicad_pcb (KiCad board)
At the start: 4 copper layers, 65 x 67 mm, 56 parts, among them J1 Conn_01x04_Pin, J10 Conn_01x06_Pin, J12 Conn_01x03_Pin, J2 Screw_Terminal_01x02, J3 Conn_01x03_Pin, J4 Conn_01x03_Pin, J5 Conn_01x04_Pin, J6 Conn_01x03_Pin, J7 Conn_01x03_Pin, J8 Conn_01x03_Pin, J9 Conn_01x03_Pin, U1 DRV8874, U2 BL9342, U3 DRV8874, U4 SN65HVD230, U5 TPS16630PWPR, U6 M95320-WMN6TP, U7 TinyThinker_J1

Commit message: added extra pins for CANBUS for daisy chaining
Parts:
- moved U6 54.0 mm to (91.1, 91.0)
- moved C14 54.0 mm to (89.7, 86.2)
- moved R15 6.97 mm to (147.8, 82.0), turned to 0 degrees
- moved J9 5.16 mm to (147.0, 79.5), turned to 180 degrees
- moved C1 0.84 mm to (143.8, 83.5)
- moved C2 0.36 mm to (141.8, 83.8)
- moved C5 0.36 mm to (139.8, 83.8)
Routing:
- net /A_IN2: track 26.5 -> 25.0 mm
- net /A_CPL: track 4.77 -> 3.52 mm
- net +BATT_PROT: track 38.2 -> 39.4 mm
- net /A_CPH: track 4.25 -> 3.39 mm
- net /A_IN1: track 27.3 -> 26.5 mm
- net GND: track 24.7 -> 24.8 mm, vias 28 -> 76
- added copper zone on F.Cu, net /A_OUT+
- added copper zone on F.Cu, net /A_OUT-
