File: pcb/DRV8874-Devboard/_autosave-DRV8874-Devboard.kicad_sch (KiCad schematic)
At the start: 56 parts, among them J1 Conn_01x04_Pin, J10 Conn_01x06_Pin, J12 Conn_01x03_Pin, J2 Screw_Terminal_01x02, J3 Conn_01x03_Pin, J4 Conn_01x03_Pin, J5 Conn_01x04_Pin, J6 Conn_01x03_Pin, J7 Conn_01x03_Pin, J8 Conn_01x03_Pin, J9 Conn_01x03_Pin, U1 DRV8874, U2 BL9342, U3 DRV8874, U4 SN65HVD230, U5 TPS16630PWPR, U6 M95320-WMN6TP, U7 TinyThinker_J1

Commit message: added extra pins for CANBUS for daisy chaining
Parts:
- U5: footprint Package_SO:HTSSOP-20-1EP_4.4x6.5mm_P0.65mm_EP2.85x4mm -> HTSSOP20_PWP_TEX
Changed lines of the file:
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@@
 			)
 		)
-		(property "Footprint" "Package_SO:HTSSOP-20-1EP_4.4x6.5mm_P0.65mm_EP2.85x4mm"
+		(property "Footprint" "HTSSOP20_PWP_TEX"
 			(at 114.3 260.35 0)
 			(effects
